File: KiCad/BMS2_2/power_module/power_module.sch (KiCad schematic (older format))
At the start: 60 parts, among them IC1 ArduinoNano, P1 BATT +, P2 BATT -, P3 72V-, P4 toRasPi, P5 FAN, Q1 CSD19535KTT, Q2 CSD19535KTT, Q3 CSD19535KTT, Q4 CSD19535KTT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

Commit message: kicad + arduino
Parts:
- C1, C11, C2, C3, C4, C6, C8, C9: symbol C -> power_module-rescue:C
- C10, C12, C13, C14, C15, C16, C17, C18, C19, C20, C21, C5, C7: symbol C_Small -> power_module-rescue:C_Small
- D1: symbol D -> power_module-rescue:D
- D2: symbol TVS -> power_module-rescue:TVS
- IC1: symbol ArduinoNano -> power_module-rescue:ArduinoNano
- L1: symbol INDUCTOR -> power_module-rescue:INDUCTOR
- P1, P2, P3: symbol CONN_01X01 -> power_module-rescue:CONN_01X01
- P4: symbol CONN_01X04 -> power_module-rescue:CONN_01X04
- P5: symbol CONN_01X02 -> power_module-rescue:CONN_01X02
- Q1, Q2, Q3, Q4: symbol Q_NMOS_GDS -> power_module-rescue:Q_NMOS_GDS
- Q5: symbol ZXMC10A816N8 -> power_module-rescue:ZXMC10A816N8
- R1, R10, R11, R12, R13, R14, R15, R16, R17, R18, R19, R2, R3, R4, R5, R6, R7, R8, R9: symbol R -> power_module-rescue:R
- U1: symbol LM5009 -> power_module-rescue:LM5009
- U2: symbol INA214 -> power_module-rescue:INA214
- U3: symbol TC1185 -> power_module-rescue:TC1185
- U4: symbol LM5112 -> power_module-rescue:LM5112
- U5: symbol SI8422 -> power_module-rescue:SI8422
- U6: symbol MAX1683 -> power_module-rescue:MAX1683
Connections:
- net GND: now also Q5.3 (S2); no longer Q5.1 (S1)
- net at C2.1, C3.1, P1.1 (P1)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: now also Q5.1 (S1); no longer Q5.3 (S2)
- net at IC1.14 (MOSI|D11): now also Q5.4 (G2); no longer Q5.2 (G1)
- net at Q5.7 (D1), Q5.8 (D1): now also R19.2; no longer Q5.4 (G2), R18.2
- net at Q5.5 (D2), Q5.6 (D2): now also Q5.2 (G1), R18.2; no longer R19.2
Other:
- moved on the sheet: R18
