File: KiCad/BMS2/Switch_matrix.sch (KiCad schematic (older format))
At the start: 124 parts, among them IC501 EMB1428Q, IC502 EMB1428Q, IC503 EMB1428Q, IC504 EMB1428Q, Q501 Q_NMOS_DGS, Q502 Q_NMOS_DGS, Q503 Q_NMOS_DGS, Q504 Q_NMOS_DGS, Q505 Q_NMOS_DGS, Q506 Q_NMOS_DGS, Q507 Q_NMOS_DGS, Q508 Q_NMOS_DGS, Q509 Q_NMOS_DGS, Q510 Q_NMOS_DGS, Q511 Q_NMOS_DGS, Q512 Q_NMOS_DGS, Q513 Q_NMOS_DGS, Q514 Q_NMOS_DGS, Q515 Q_NMOS_DGS, Q516 Q_NMOS_DGS, Q517 Q_NMOS_DGS, Q518 Q_NMOS_DGS, Q519 Q_NMOS_DGS, Q520 Q_NMOS_DGS, Q521 Q_NMOS_DGS, Q522 Q_NMOS_DGS, Q523 Q_NMOS_DGS, Q524 Q_NMOS_DGS, Q525 Q_NMOS_DGS, Q526 Q_NMOS_DGS, Q527 Q_NMOS_DGS, Q528 Q_NMOS_DGS, Q529 Q_NMOS_DGS, Q530 Q_NMOS_DGS, Q531 Q_NMOS_DGS, Q532 Q_NMOS_DGS, Q533 Q_NMOS_DGS, Q534 Q_NMOS_DGS, Q535 Q_NMOS_DGS, Q536 Q_NMOS_DGS, Q537 Q_NMOS_DGS, Q538 Q_NMOS_DGS, Q539 Q_NMOS_DGS, Q540 Q_NMOS_DGS, Q541 Q_NMOS_DGS, Q542 Q_NMOS_DGS, Q543 Q_NMOS_DGS, Q544 Q_NMOS_DGS, Q545 Q_NMOS_DGS, Q546 Q_NMOS_DGS, Q547 Q_NMOS_DGS, Q548 Q_NMOS_DGS, Q549 Q_NMOS_DGS, Q550 Q_NMOS_DGS, Q551 Q_NMOS_DGS, Q552 Q_NMOS_DGS, Q553 Q_NMOS_DGS, Q554 Q_NMOS_DGS, Q555 Q_NMOS_DGS, Q556 Q_NMOS_DGS, Q557 Q_NMOS_DGS, Q558 Q_NMOS_DGS, Q559 Q_NMOS_DGS, Q560 Q_NMOS_DGS, Q561 Q_NMOS_DGS, Q562 Q_NMOS_DGS, Q563 Q_NMOS_DGS, Q564 Q_NMOS_DGS, Q565 Q_NMOS_DGS, Q566 Q_NMOS_DGS, Q567 Q_NMOS_DGS, Q568 Q_NMOS_DGS, Q569 Q_NMOS_DGS, Q570 Q_NMOS_DGS, Q571 Q_NMOS_DGS, Q572 Q_NMOS_DGS, Q573 Q_NMOS_DGS, Q574 Q_NMOS_DGS, Q575 Q_NMOS_DGS, Q576 Q_NMOS_DGS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

Commit message: Added slides for all entries
All entries are now derived from Entry -class
Parts:
- C501, C502, C503, C504, C505, C506, C507, C508, C509, C510, C511, C512: symbol C -> Device:C
- D501, D502, D503, D504, D505, D506, D507, D508, D509, D510, D511, D512, D513, D514, D515, D516, D517, D518, D519, D520: symbol D -> Device:D
- IC501, IC502, IC503, IC504: symbol EMB1428Q -> EMB1428Q:EMB1428Q
- Q501, Q502, Q503, Q504, Q505, Q506, Q507, Q508, Q509, Q510, Q511, Q512, Q513, Q514, Q515, Q516, Q517, Q518, Q519, Q520, Q521, Q522, Q523, Q524, Q525, Q526, Q527, Q528, Q529, Q530, Q531, Q532, Q533, Q534, Q535, Q536, Q537, Q538, Q539, Q540, Q541, Q542, Q543, Q544, Q545, Q546, Q547, Q548, Q549, Q550, Q551, Q552, Q553, Q554, Q555, Q556, Q557, Q558, Q559, Q560, Q561, Q562, Q563, Q564, Q565, Q566, Q567, Q568, Q569, Q570, Q571, Q572, Q573, Q574, Q575, Q576, Q577, Q578, Q579, Q580: symbol Q_NMOS_DGS -> Device:Q_NMOS_DGS
- R501, R502, R503, R504: symbol R -> Device:R
- U501, U503: symbol ISO7342FC -> texas:ISO7342FC
- U502, U504: symbol ISO7341FC -> texas:ISO7341FC
